File: SolderProject.kicad_sch (KiCad schematic)
At the start: 18 parts, among them U1 NE555P, U2 4017

Commit message: V1
Other:
- note removed: "TODO: - Silkscreen: - IEEE Logo for LEDs - IEEE club QR code - Board Github QR code - component selection"
- title: (none) -> Solder Project
Changed lines of the file:
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@@
 (kicad_sch (version 20211123) (generator eeschema)
   (paper "A5")
+  (title_block
+    (title "Solder Project")
+    (comment 1 "By Zane C")
+  )
   (junction (at 151.13 67.31) (diameter 0) (color 0 0 0 0)
   )
@@
     (stroke (width 0) (type default) (color 0 0 0 0))
   )
-  (text "TODO:\n - Silkscreen:\n    - IEEE Logo for LEDs\n    - IEEE club QR code\n    - Board Github QR code\n - component selection\n"
-    (at 144.78 34.29 0)
-    (effects (font (size 1.27 1.27)) (justify left bottom))
-  )
   (label "LED_K" (at 151.13 74.93 0)

Commit message: V1.1 - Slight improvements VMax changed to 14V
Parts:
- B1: value 5V-15V -> 5V-14V
Changed lines of the file:
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@@
       (effects (font (size 1.27 1.27)) (justify left))
     )
-    (property "Value" "5V-15V" (id 1) (at 26.67 61.4679 0)
+    (property "Value" "5V-14V" (id 1) (at 26.67 61.4679 0)
       (effects (font (size 1.27 1.27)) (justify left))
     )
@@
     )
     (path "/593f335d-d488-4988-85df-238b218b998e"
-      (reference "B1") (unit 1) (value "5V-15V") (footprint "Connector_PinHeader_2.54mm:PinHeader_1x02_P2.54mm_Vertical")
+      (reference "B1") (unit 1) (value "5V-14V") (footprint "Connector_PinHeader_2.54mm:PinHeader_1x02_P2.54mm_Vertical")
     )
     (path "/54874b9c-f3e3-4955-9dfb-de4fec668e9d"
